File: currentscaler/currentscaler.sch (KiCad schematic (older format))
At the start: 35 parts

Commit message: temp commit
Parts:
- added U?: MAX4238AUT, Package_TO_SOT_SMD:SOT-23-6, symbol Amplifier_Operational:MAX4238AUT
- C1, C2, C3, C4, C5, C6, C7: renamed from C?; footprint (none) -> Capacitor_SMD:C_0402_1005Metric
- R1, R10, R11, R12, R13, R14, R15, R2, R3, R4, R5, R6, R7, R8, R9: renamed from R?; footprint (none) -> Resistor_SMD:R_0402_1005Metric
- TP1, TP2, TP3, TP4: renamed from TP?; footprint (none) -> Connector:Banana_Jack_1Pin
- U1, U2, U3: renamed from U?; footprint (none) -> Package_TO_SOT_SMD:SOT-23-5
- gave numbers to parts that had none: 6

Commit message: Started PCB
Designing for Hammond 1550Q.
Parts:
- removed C5: 10p, Capacitor_SMD:C_0402_1005Metric, symbol Device:C_Small
- removed C6: 100nF, Capacitor_SMD:C_0402_1005Metric, symbol Device:C_Small
- removed JP1, JP3: SolderJumper_3_Bridged12, symbol Jumper:SolderJumper_3_Bridged12
- removed JP2: SolderJumper_2_Open, symbol Jumper:SolderJumper_2_Open
- removed Q1, Q2: Q_PMOS_DGS, symbol Device:Q_PMOS_DGS
- removed R11: 1k .05%, Resistor_SMD:R_0402_1005Metric, symbol Device:R_Small
- removed R12: 6.8k .05%, Resistor_SMD:R_0402_1005Metric, symbol Device:R_Small
- removed R13: 2.2k .05%, Resistor_SMD:R_0402_1005Metric, symbol Device:R_Small
- removed U1, U2, U3: OPA189, Package_TO_SOT_SMD:SOT-23-5, symbol athir:OPA189
- added C1: 100uF, Capacitor_SMD:CP_Elec_6.3x7.7, symbol Device:CP_Small
- added C2: 100nF, Capacitor_SMD:C_0402_1005Metric, symbol Device:C_Small
- added J1: USB_B, Connector_USB:USB_Micro-B_Molex_47346-0001, symbol Connector:USB_B
- added Q1, Q2: NTR5103NT1G, Package_TO_SOT_SMD:SOT-23, symbol athir:NTR5103NT1G
- added SW1: SW_SP3T, Connector_PinHeader_2.54mm:PinHeader_1x04_P2.54mm_Vertical, symbol Switch:SW_SP3T
- added SW2: SW_SPST, Connector_PinHeader_2.54mm:PinHeader_1x02_P2.54mm_Vertical, symbol Switch:SW_SPST
- added U2: MAX4238AUT, Package_SO:SO-8_5.3x6.2mm_P1.27mm, symbol Amplifier_Operational:MAX4239ASA
- TP1, TP2, TP3, TP4: footprint Connector:Banana_Jack_1Pin -> TestPoint:TestPoint_THTPad_D4.0mm_Drill2.0mm
- U1: renamed from U?; footprint Package_TO_SOT_SMD:SOT-23-6 -> Package_SO:SO-8_5.3x6.2mm_P1.27mm; symbol Amplifier_Operational:MAX4238AUT -> Amplifier_Operational:MAX4239ASA
- renumbered C1 to C3, C2 to C4, C3 to C5, C4 to C6, R14 to R11, R15 to R12
Connections:
- net labels removed: +12V
- wire segments 117 -> 105
- no-connect marks 0 -> 3

Commit message: HW: rev 1 - Gerbers
Parts:
- removed C1: 100uF, Capacitor_SMD:CP_Elec_6.3x7.7, symbol Device:CP_Small
- removed C7: 100nF, Capacitor_SMD:C_0402_1005Metric, symbol Device:C_Small
- removed J1: USB_B, Connector_USB:USB_Micro-B_Molex_47346-0001, symbol Connector:USB_B
- removed Q1, Q2: NTR5103NT1G, Package_TO_SOT_SMD:SOT-23, symbol athir:NTR5103NT1G
- removed Q3: BC817, Package_TO_SOT_SMD:SOT-23, symbol Transistor_BJT:BC817
- removed SW1: SW_SP3T, Connector_PinHeader_2.54mm:PinHeader_1x04_P2.54mm_Vertical, symbol Switch:SW_SP3T
- removed SW2: SW_SPST, Connector_PinHeader_2.54mm:PinHeader_1x02_P2.54mm_Vertical, symbol Switch:SW_SPST
- removed U1, U2: MAX4238AUT, Package_SO:SO-8_5.3x6.2mm_P1.27mm, symbol Amplifier_Operational:MAX4239ASA
- added BT1: Battery_Cell, Battery:BatteryHolder_Keystone_3008_1x2450, symbol Device:Battery_Cell
- added C1: 100nF, Capacitor_SMD:C_0603_1608Metric, symbol Device:C_Small
- added DP3T1: OS203013MT6QN1, athir:OS203013MT6QN1, symbol athir:OS203013MT6QN1
- added R13: 2.2k .05%, Resistor_SMD:R_0603_1608Metric, symbol Device:R_Small
- added R14: 100, Resistor_SMD:R_0603_1608Metric, symbol Device:R_Small
- added U1: LMV321, Package_TO_SOT_SMD:SOT-23-5, symbol Amplifier_Operational:LMV321
- added U2, U3: MAX4239AUT, Package_TO_SOT_SMD:SOT-23-6, symbol Amplifier_Operational:MAX4239AUT
- C2, C4: value 100nF -> 10p; footprint Capacitor_SMD:C_0402_1005Metric -> Capacitor_SMD:C_0603_1608Metric
- C3, C5: value 10p -> 100nF; footprint Capacitor_SMD:C_0402_1005Metric -> Capacitor_SMD:C_0603_1608Metric
- C6: footprint Capacitor_SMD:C_0402_1005Metric -> Capacitor_SMD:C_0603_1608Metric
- R1, R10, R9: footprint Resistor_SMD:R_0402_1005Metric -> Resistor_SMD:R_0603_1608Metric
- R11: value 10k -> 1k .05%; footprint Resistor_SMD:R_0402_1005Metric -> Resistor_SMD:R_0603_1608Metric
- R12: value 220 -> 6.8k .05%; footprint Resistor_SMD:R_0402_1005Metric -> Resistor_SMD:R_0603_1608Metric
- R2: value 10 .05% -> 100k 1%; footprint Resistor_SMD:R_0402_1005Metric -> Resistor_SMD:R_0603_1608Metric
- R3: value 10m .05% -> 100k 1%; footprint Resistor_SMD:R_0402_1005Metric -> Resistor_SMD:R_0603_1608Metric
- R4: value 220 -> 10m .05%; footprint Resistor_SMD:R_0402_1005Metric -> Resistor_SMD:R_0603_1608Metric
- R5: value 1k .05% -> 10 .05%; footprint Resistor_SMD:R_0402_1005Metric -> Resistor_SMD:R_0603_1608Metric
- R6: value 6.8k .05% -> 100; footprint Resistor_SMD:R_0402_1005Metric -> Resistor_SMD:R_0603_1608Metric
- R7: value 2.2k .05% -> 1k .05%; footprint Resistor_SMD:R_0402_1005Metric -> Resistor_SMD:R_0603_1608Metric
- R8: value 1k .05% -> 100; footprint Resistor_SMD:R_0402_1005Metric -> Resistor_SMD:R_0603_1608Metric
- TP1: value SOURCE -> IN_P
- TP2: value LOAD -> IN_N
- TP3: value VOUT -> OUT_P
- TP4: value GND -> OUT_N
Connections:
- net labels added: +9V, GNDREF
- net labels removed: LP_EN, VCC, mEN, uEN
- wire segments 105 -> 110
- no-connect marks 3 -> 1
Other:
- note added: "CHANGE TO MAX44246 TO SUPPORT 9V"

Commit message: HW: rev 2 - Gerbers
Corrected DP3T footprint.
Added 3D file for entire PCB.
Parts:
- removed TP1: IN_P, TestPoint:TestPoint_THTPad_D4.0mm_Drill2.0mm, symbol Connector:TestPoint
- removed TP2: IN_N, TestPoint:TestPoint_THTPad_D4.0mm_Drill2.0mm, symbol Connector:TestPoint
- removed TP3: OUT_P, TestPoint:TestPoint_THTPad_D4.0mm_Drill2.0mm, symbol Connector:TestPoint
- removed TP4: OUT_N, TestPoint:TestPoint_THTPad_D4.0mm_Drill2.0mm, symbol Connector:TestPoint
- added CON1, CON2: RS677-8759, athir:6778759, symbol athir:RS677-8759
Connections:
- wire segments 110 -> 114
Changed lines of the file:
@@
 	9700 4450 9350 4450
 Wire Wire Line
-	9700 4450 9800 4450
+	9700 4450 10200 4450
 Connection ~ 9700 4450
 Wire Wire Line
-	9700 5900 9825 5900
-$Comp
-L Connector:TestPoint TP3
-U 1 1 5CAAF213
-P 9800 4450
-AR Path="/5CAAF213" Ref="TP3"  Part="1"
-AR Path="/5C9A6AC0/5CAAF213" Ref="TP?"  Part="1"
-F 0 "TP3" V 9754 4637 50  0000 L CNN
-F 1 "OUT_P" V 9845 4637 50  0000 L CNN
-F 2 "TestPoint:TestPoint_THTPad_D4.0mm_Drill2.0mm" H 10000 4450 50  0001 C CNN
-F 3 "~" H 10000 4450 50  0001 C CNN
-	1    9800 4450
-	0    1    1    0
-$EndComp
-$Comp
-L Connector:TestPoint TP4
-U 1 1 5CAAF21A
-P 9825 5900
-AR Path="/5CAAF21A" Ref="TP4"  Part="1"
-AR Path="/5C9A6AC0/5CAAF21A" Ref="TP?"  Part="1"
-F 0 "TP4" V 9779 6087 50  0000 L CNN
-F 1 "OUT_N" V 9870 6087 50  0000 L CNN
-F 2 "TestPoint:TestPoint_THTPad_D4.0mm_Drill2.0mm" H 10025 5900 50  0001 C CNN
-F 3 "~" H 10025 5900 50  0001 C CNN
-	1    9825 5900
-	0    1    1    0
-$EndComp
+	9700 5900 10200 5900
 Wire Wire Line
 	7550 4450 9150 4450
@@
 Wire Wire Line
 	5425 4375 5275 4375
-$Comp
-L Connector:TestPoint TP1
-U 1 1 5CAAF242
-P 1050 3550
-AR Path="/5CAAF242" Ref="TP1"  Part="1"
-AR Path="/5C9A6AC0/5CAAF242" Ref="TP?"  Part="1"
-F 0 "TP1" V 1245 3624 50  0000 C CNN
-F 1 "IN_P" V 1154 3624 50  0000 C CNN
-F 2 "TestPoint:TestPoint_THTPad_D4.0mm_Drill2.0mm" H 1250 3550 50  0001 C CNN
-F 3 "~" H 1250 3550 50  0001 C CNN
-	1    1050 3550
-	0    -1   -1   0
-$EndComp
-$Comp
-L Connector:TestPoint TP2
-U 1 1 5CAAF249
-P 1075 5150
-AR Path="/5CAAF249" Ref="TP2"  Part="1"
-AR Path="/5C9A6AC0/5CAAF249" Ref="TP?"  Part="1"
-F 0 "TP2" V 1270 5224 50  0000 C CNN
-F 1 "IN_N" V 1179 5224 50  0000 C CNN
-F 2 "TestPoint:TestPoint_THTPad_D4.0mm_Drill2.0mm" H 1275 5150 50  0001 C CNN
-F 3 "~" H 1275 5150 50  0001 C CNN
-	1    1075 5150
-	0    -1   -1   0
-$EndComp
 Connection ~ 4900 5900
 Wire Wire Line
@@
 	1375 3550 1375 3650
 Wire Wire Line
-	1050 3550 1375 3550
-Wire Wire Line
 	1375 5150 1850 5150
 Wire Wire Line
@@
 	2050 3425 2050 3775
 Connection ~ 2050 3775
-Wire Wire Line
-	1075 5150 1375 5150
 Connection ~ 1375 5150
 Wire Wire Line
@@
 Text Notes 5625 1500 0    50   ~ 0
 CHANGE TO MAX44246 TO SUPPORT 9V
+$Comp
+L athir:RS677-8759 CON1
+U 1 1 5C9E8BAB
+P 925 4300
+F 0 "CON1" H 1003 4346 50  0000 L CNN
+F 1 "RS677-8759" H 1003 4255 50  0000 L CNN
+F 2 "athir:6778759" H 925 4300 50  0001 C CNN
+F 3 "" H 925 4300 50  0001 C CNN
+	1    925  4300
+	1    0    0    -1
+$EndComp
+$Comp
+L athir:RS677-8759 CON2
+U 1 1 5C9E8C1B
+P 10200 5150
+F 0 "CON2" H 10278 5196 50  0000 L CNN
+F 1 "RS677-8759" H 10278 5105 50  0000 L CNN
+F 2 "athir:6778759" H 10200 5150 50  0001 C CNN
+F 3 "" H 10200 5150 50  0001 C CNN
+	1    10200 5150
+	1    0    0    -1
+$EndComp
+Wire Wire Line
+	10200 5500 10200 5900
+Wire Wire Line
+	10200 4800 10200 4450
+Wire Wire Line
+	925  3950 925  3550
+Wire Wire Line
+	925  3550 1375 3550
+Wire Wire Line
+	925  4650 925  5150
+Wire Wire Line
+	925  5150 1375 5150
 $EndSCHEMATC

Commit message: WIP: HW4
100 ohm resistors now 0805.
Fixed footprint of switch.
Removed 3V CR2450 holder.
Added silkscreen explanations.
Parts:
- BT1: footprint Battery:BatteryHolder_Keystone_3008_1x2450 -> Resistor_SMD:R_4020_10251Metric
- R14, R6, R8: footprint Resistor_SMD:R_0603_1608Metric -> Resistor_SMD:R_0805_2012Metric
Connections:
- net labels added: +5V
- net labels removed: +9V
- wire segments 114 -> 121
Changed lines of the file:
@@
 EESchema Schematic File Version 4
 LIBS:currentscaler-cache
-EELAYER 26 0
+EELAYER 29 0
 EELAYER END
 $Descr A4 11693 8268
@@
 AR Path="/5CAAF185" Ref="U3"  Part="1"
 F 0 "U3" H 7516 4496 50  0000 L CNN
-F 1 "MAX4239AUT" H 7516 4405 50  0000 L CNN
+F 1 "MAX4239AUT" H 7600 4400 50  0000 L CNN
 F 2 "Package_TO_SOT_SMD:SOT-23-6" H 7175 4450 50  0001 C CNN
 F 3 "http://datasheets.maximintegrated.com/en/ds/MAX4238-MAX4239.pdf" H 7325 4600 50  0001 C CNN
@@
 AR Path="/5CAAF1BF" Ref="U2"  Part="1"
 F 0 "U2" H 6066 4521 50  0000 L CNN
-F 1 "MAX4239AUT" H 6066 4430 50  0000 L CNN
+F 1 "MAX4239AUT" H 6175 4425 50  0000 L CNN
 F 2 "Package_TO_SOT_SMD:SOT-23-6" H 5725 4475 50  0001 C CNN
 F 3 "http://datasheets.maximintegrated.com/en/ds/MAX4238-MAX4239.pdf" H 5875 4625 50  0001 C CNN
@@
 F 0 "R14" V 9054 4450 50  0000 C CNN
 F 1 "100" V 9145 4450 50  0000 C CNN
-F 2 "Resistor_SMD:R_0603_1608Metric" H 9250 4450 50  0001 C CNN
+F 2 "Resistor_SMD:R_0805_2012Metric" H 9250 4450 50  0001 C CNN
 F 3 "~" H 9250 4450 50  0001 C CNN
 	1    9250 4450
@@
 F 0 "R6" V 3079 5900 50  0000 C CNN
 F 1 "100" V 3170 5900 50  0000 C CNN
-F 2 "Resistor_SMD:R_0603_1608Metric" H 3275 5900 50  0001 C CNN
+F 2 "Resistor_SMD:R_0805_2012Metric" H 3275 5900 50  0001 C CNN
 F 3 "~" H 3275 5900 50  0001 C CNN
 	1    3275 5900
@@
 F 0 "R8" V 4979 4375 50  0000 C CNN
 F 1 "100" V 5070 4375 50  0000 C CNN
-F 2 "Resistor_SMD:R_0603_1608Metric" H 5175 4375 50  0001 C CNN
+F 2 "Resistor_SMD:R_0805_2012Metric" H 5175 4375 50  0001 C CNN
 F 3 "~" H 5175 4375 50  0001 C CNN
 	1    5175 4375
@@
 Wire Wire Line
 	1650 6100 1650 6375
-$Comp
-L power:+9V #PWR?
-U 1 1 5CAAF2AA
-P 1650 5500
-AR Path="/5C9A6AC0/5CAAF2AA" Ref="#PWR?"  Part="1"
-AR Path="/5CAAF2AA" Ref="#PWR0103"  Part="1"
-F 0 "#PWR0103" H 1650 5350 50  0001 C CNN
-F 1 "+9V" H 1665 5673 50  0000 C CNN
-F 2 "" H 1650 5500 50  0001 C CNN
-F 3 "" H 1650 5500 50  0001 C CNN
-	1    1650 5500
-	1    0    0    -1
-$EndComp
 Wire Wire Line
 	1650 5500 1650 5575
@@
 Wire Wire Line
 	2875 5475 2725 5475
-$Comp
-L power:+9V #PWR?
-U 1 1 5CAAF2DA
-P 2425 5400
-AR Path="/5C9A6AC0/5CAAF2DA" Ref="#PWR?"  Part="1"
-AR Path="/5CAAF2DA" Ref="#PWR0108"  Part="1"
-F 0 "#PWR0108" H 2425 5250 50  0001 C CNN
-F 1 "+9V" H 2440 5573 50  0000 C CNN
-F 2 "" H 2425 5400 50  0001 C CNN
-F 3 "" H 2425 5400 50  0001 C CNN
-	1    2425 5400
-	1    0    0    -1
-$EndComp
 Wire Wire Line
 	2425 5400 2425 5475
@@
 Wire Wire Line
 	5625 4850 5625 4775
-$Comp
-L power:+9V #PWR?
-U 1 1 5CAAF2E3
-P 5625 3975
-AR Path="/5C9A6AC0/5CAAF2E3" Ref="#PWR?"  Part="1"
-AR Path="/5CAAF2E3" Ref="#PWR0109"  Part="1"
-F 0 "#PWR0109" H 5625 3825 50  0001 C CNN
-F 1 "+9V" H 5640 4148 50  0000 C CNN
-F 2 "" H 5625 3975 50  0001 C CNN
-F 3 "" H 5625 3975 50  0001 C CNN
-	1    5625 3975
-	1    0    0    -1
-$EndComp
 Wire Wire Line
 	5625 3975 5625 4050
@@
 Wire Wire Line
 	7075 3975 7075 4150
-$Comp
-L power:+9V #PWR?
-U 1 1 5CAAF30D
-P 7075 3925
-AR Path="/5C9A6AC0/5CAAF30D" Ref="#PWR?"  Part="1"
-AR Path="/5CAAF30D" Ref="#PWR0112"  Part="1"
-F 0 "#PWR0112" H 7075 3775 50  0001 C CNN
-F 1 "+9V" H 7090 4098 50  0000 C CNN
-F 2 "" H 7075 3925 50  0001 C CNN
-F 3 "" H 7075 3925 50  0001 C CNN
-	1    7075 3925
-	1    0    0    -1
-$EndComp
 Wire Wire Line
 	7075 3925 7075 3975
@@
 F 0 "BT1" H 5043 1971 50  0000 L CNN
 F 1 "Battery_Cell" H 5043 1880 50  0000 L CNN
-F 2 "Battery:BatteryHolder_Keystone_3008_1x2450" V 4925 1935 50  0001 C CNN
+F 2 "Resistor_SMD:R_4020_10251Metric" V 4925 1935 50  0001 C CNN
 F 3 "~" V 4925 1935 50  0001 C CNN
 	1    4925 1875
@@
 Wire Wire Line
 	4925 1975 4925 2050
-$Comp
-L power:+9V #PWR0114
-U 1 1 5CAB9E8D
-P 4925 1575
-F 0 "#PWR0114" H 4925 1425 50  0001 C CNN
-F 1 "+9V" H 4940 1748 50  0000 C CNN
-F 2 "" H 4925 1575 50  0001 C CNN
-F 3 "" H 4925 1575 50  0001 C CNN
-	1    4925 1575
-	1    0    0    -1
-$EndComp
 Wire Wire Line
 	4925 1575 4925 1675
@@
 Wire Wire Line
 	925  5150 1375 5150
+Wire Wire Line
+	5900 4775 5900 4800
+Wire Wire Line
+	5900 4800 5725 4800
+Wire Wire Line
+	5725 4800 5725 4775
+Wire Wire Line
+	7350 4750 7350 4800
+Wire Wire Line
+	7350 4800 7175 4800
+Wire Wire Line
+	7175 4800 7175 4750
+$Comp
+L power:PWR_FLAG #FLG0101
+U 1 1 5CE2B498
+P 7100 1925
+F 0 "#FLG0101" H 7100 2000 50  0001 C CNN
+F 1 "PWR_FLAG" H 7100 2099 50  0000 C CNN
+F 2 "" H 7100 1925 50  0001 C CNN
+F 3 "~" H 7100 1925 50  0001 C CNN
+	1    7100 1925
+	1    0    0    -1
+$EndComp
+Wire Wire Line
+	7100 1925 7100 2275
+$Comp
+L power:+5V #PWR0103
+U 1 1 5CE3122B
+P 2425 5400
+F 0 "#PWR0103" H 2425 5250 50  0001 C CNN
+F 1 "+5V" H 2440 5573 50  0000 C CNN
+F 2 "" H 2425 5400 50  0001 C CNN
+F 3 "" H 2425 5400 50  0001 C CNN
+	1    2425 5400
+	1    0    0    -1
+$EndComp
+$Comp
+L power:+5V #PWR0108
+U 1 1 5CE31F4E
+P 5625 3975
+F 0 "#PWR0108" H 5625 3825 50  0001 C CNN
+F 1 "+5V" H 5640 4148 50  0000 C CNN
+F 2 "" H 5625 3975 50  0001 C CNN
+F 3 "" H 5625 3975 50  0001 C CNN
+	1    5625 3975
+	1    0    0    -1
+$EndComp
+$Comp
+L power:+5V #PWR0109
+U 1 1 5CE32F15
+P 7075 3925
+F 0 "#PWR0109" H 7075 3775 50  0001 C CNN
+F 1 "+5V" H 7090 4098 50  0000 C CNN
+F 2 "" H 7075 3925 50  0001 C CNN
+F 3 "" H 7075 3925 50  0001 C CNN
+	1    7075 3925
+	1    0    0    -1
+$EndComp
+$Comp
+L power:+5V #PWR0112
+U 1 1 5CE33C48
+P 7100 2275
+F 0 "#PWR0112" H 7100 2125 50  0001 C CNN
+F 1 "+5V" H 7115 2448 50  0000 C CNN
+F 2 "" H 7100 2275 50  0001 C CNN
+F 3 "" H 7100 2275 50  0001 C CNN
+	1    7100 2275
+	-1   0    0    1
+$EndComp
+$Comp
+L power:+5V #PWR0114
+U 1 1 5CE34C46
+P 4925 1575
+F 0 "#PWR0114" H 4925 1425 50  0001 C CNN
+F 1 "+5V" H 4940 1748 50  0000 C CNN
+F 2 "" H 4925 1575 50  0001 C CNN
+F 3 "" H 4925 1575 50  0001 C CNN
+	1    4925 1575
+	1    0    0    -1
+$EndComp
+$Comp
+L power:+5V #PWR0117
+U 1 1 5CE38469
+P 1650 5500
+F 0 "#PWR0117" H 1650 5350 50  0001 C CNN
+F 1 "+5V" H 1665 5673 50  0000 C CNN
+F 2 "" H 1650 5500 50  0001 C CNN
+F 3 "" H 1650 5500 50  0001 C CNN
+	1    1650 5500
+	1    0    0    -1
+$EndComp
+$Comp
+L power:+5V #PWR0115
+U 1 1 5CE39B28
+P 7350 4750
+F 0 "#PWR0115" H 7350 4600 50  0001 C CNN
+F 1 "+5V" H 7365 4923 50  0000 C CNN
+F 2 "" H 7350 4750 50  0001 C CNN
+F 3 "" H 7350 4750 50  0001 C CNN
+	1    7350 4750
+	1    0    0    -1
+$EndComp
+$Comp
+L power:+5V #PWR0116
+U 1 1 5CE3AC0F
+P 5900 4775
+F 0 "#PWR0116" H 5900 4625 50  0001 C CNN
+F 1 "+5V" H 5915 4948 50  0000 C CNN
+F 2 "" H 5900 4775 50  0001 C CNN
+F 3 "" H 5900 4775 50  0001 C CNN
+	1    5900 4775
+	1    0    0    -1
+$EndComp
 $EndSCHEMATC

Commit message: HW 4 - commit
Parts:
- added C7: 100nF, Capacitor_SMD:C_0603_1608Metric, symbol Device:C_Small
- added U4: MAX44246, athir:uMAX8, symbol athir:MAX44246
Connections:
- wire segments 121 -> 148
Changed lines of the file:
@@
 	6550 4350 6550 4475
 Wire Wire Line
-	6550 4475 6100 4475
+	6550 4475 6350 4475
 Connection ~ 6100 4475
 Wire Wire Line
@@
 	9700 5900 10200 5900
 Wire Wire Line
-	7550 4450 9150 4450
+	7550 4450 8125 4450
 Connection ~ 7550 4450
 Wire Wire Line
@@
 $EndComp
 Wire Wire Line
-	5425 4375 5275 4375
+	5425 4375 5350 4375
 Connection ~ 4900 5900
 Wire Wire Line
@@
 	1    0    0    -1
 $EndComp
+$Comp
+L athir:MAX44246 U4
+U 1 1 5CF03F30
+P 6375 3175
+F 0 "U4" H 6500 3640 50  0000 C CNN
+F 1 "MAX44246" H 6500 3549 50  0000 C CNN
+F 2 "athir:uMAX8" H 6375 3175 50  0001 C CNN
+F 3 "" H 6375 3175 50  0001 C CNN
+	1    6375 3175
+	1    0    0    -1
+$EndComp
+Wire Wire Line
+	6050 3275 6050 3350
+Wire Wire Line
+	6050 3275 6125 3275
+Wire Wire Line
+	6125 3175 5350 3175
+Wire Wire Line
+	5350 3175 5350 4375
+Connection ~ 5350 4375
+Wire Wire Line
+	5350 4375 5275 4375
+Wire Wire Line
+	6125 3075 4975 3075
+Wire Wire Line
+	4975 3075 4975 4575
+Wire Wire Line
+	4975 4575 5325 4575
+Connection ~ 5325 4575
+Wire Wire Line
+	6125 2975 5875 2975
+Wire Wire Line
+	5875 2975 5875 3575
+Wire Wire Line
+	5875 3575 6350 3575
+Wire Wire Line
+	6950 3575 6950 3275
+Wire Wire Line
+	6950 3275 6875 3275
+Wire Wire Line
+	6350 3575 6350 4475
+Connection ~ 6350 3575
+Wire Wire Line
+	6350 3575 6950 3575
+Connection ~ 6350 4475
+Wire Wire Line
+	6350 4475 6100 4475
+Wire Wire Line
+	6875 3175 7025 3175
+Wire Wire Line
+	7025 3175 7025 3675
+Wire Wire Line
+	7025 3675 6675 3675
+Wire Wire Line
+	6675 3675 6675 4550
+Wire Wire Line
+	6675 4550 6775 4550
+Connection ~ 6775 4550
+Wire Wire Line
+	6875 3075 8125 3075
+Wire Wire Line
+	8125 3075 8125 4450
+Connection ~ 8125 4450
+Wire Wire Line
+	8125 4450 9150 4450
+$Comp
+L Device:C_Small C7
+U 1 1 5CF2FFED
+P 7100 2975
+AR Path="/5CF2FFED" Ref="C7"  Part="1"
+AR Path="/5C9A6AC0/5CF2FFED" Ref="C?"  Part="1"
+F 0 "C7" V 6871 2975 50  0000 C CNN
+F 1 "100nF" V 6962 2975 50  0000 C CNN
+F 2 "Capacitor_SMD:C_0603_1608Metric" H 7100 2975 50  0001 C CNN
+F 3 "~" H 7100 2975 50  0001 C CNN
+	1    7100 2975
+	0    1    1    0
+$EndComp
+Wire Wire Line
+	7000 2975 6875 2975
+$Comp
+L power:GND #PWR?
+U 1 1 5CF36EC3
+P 7250 3175
+AR Path="/5C9A6AC0/5CF36EC3" Ref="#PWR?"  Part="1"
+AR Path="/5CF36EC3" Ref="#PWR0118"  Part="1"
+F 0 "#PWR0118" H 7250 2925 50  0001 C CNN
+F 1 "GND" H 7255 3002 50  0000 C CNN
+F 2 "" H 7250 3175 50  0001 C CNN
+F 3 "" H 7250 3175 50  0001 C CNN
+	1    7250 3175
+	1    0    0    -1
+$EndComp
+Wire Wire Line
+	7250 3175 7250 2975
+Wire Wire Line
+	7250 2975 7200 2975
+$Comp
+L power:GND #PWR0119
+U 1 1 5CF3D8DD
+P 6050 3350
+AR Path="/5CF3D8DD" Ref="#PWR0119"  Part="1"
+AR Path="/5C9A6AC0/5CF3D8DD" Ref="#PWR?"  Part="1"
+F 0 "#PWR0119" H 6050 3100 50  0001 C CNN
+F 1 "GND" H 6055 3177 50  0000 C CNN
+F 2 "" H 6050 3350 50  0001 C CNN
+F 3 "" H 6050 3350 50  0001 C CNN
+	1    6050 3350
+	1    0    0    -1
+$EndComp
